Commit message: save map; add arm; nav vis

File: unitree_ros-master/robots/aliengo_description/xacro/aliengo.urdf (robot description, URDF)
Before this commit: robot aliengo_description, 29 links, 28 joints
Links:
- added link bottom_link, mass 0.2; collision box size=0.1 0.1 0.01; visual box size=0.1 0.1 0.01
- added link grasping_frame
- added link gripper_finger_link1, mass 0.2; visual box size=0.08 0.01 0.01
- added link gripper_finger_link2, mass 0.2; visual box size=0.08 0.01 0.01
- added link link1, mass 0.2; collision cylinder length=0.15 radius=0.03; visual cylinder length=0.15 radius=0.03
- added link link2, mass 0.2; collision cylinder length=0.22 radius=0.03; visual cylinder length=0.22 radius=0.03
- added link link3, mass 0.2; collision cylinder length=0.14 radius=0.03; visual cylinder length=0.14 radius=0.03
- added link link4, mass 0.2; collision cylinder length=0.03 radius=0.025; visual cylinder length=0.03 radius=0.025
- added link link5, mass 0.2; collision cylinder length=0.06 radius=0.03; visual cylinder length=0.06 radius=0.03
- added link link6, mass 0.2; collision cylinder length=0.02 radius=0.04; visual cylinder length=0.02 radius=0.04
Joints:
- added joint bottom_joint: type fixed, parent trunk, child bottom_link, origin xyz=0 0 0 rpy=0 0 0
- added joint finger_joint1: type prismatic, parent link6, child gripper_finger_link1, origin xyz=0.0 0 0, axis 0 1 0, limit lower=0 upper=0.015 effort=100 velocity=0.05
- added joint finger_joint2: type prismatic, parent link6, child gripper_finger_link2, origin xyz=0.0 0 0, axis 0 -1 0, limit lower=0 upper=0.015 effort=100 velocity=0.05
- added joint grasping_frame_joint: type fixed, parent link6, child grasping_frame, origin xyz=0.08 0 0 rpy=0 0 0
- added joint joint1: type revolute, parent trunk, child link1, origin xyz=0 0 0.02 rpy=0 1.570795 0, axis -1 0 0, limit lower=-2.96 upper=2.96 effort=300 velocity=1
- added joint joint2: type revolute, parent link1, child link2, origin xyz=-0.15 0 0.0 rpy=-1.570795 0 1.570795, axis 1 0 0, limit lower=-2.35 upper=2.35 effort=300 velocity=1
- added joint joint3: type revolute, parent link2, child link3, origin xyz=0 0 0.22 rpy=0 3.14159 0, axis -1 0 0, limit lower=-2.62 upper=2.62 effort=300 velocity=1
- added joint joint4: type revolute, parent link3, child link4, origin xyz=0.0 0.0 -0.14 rpy=0 1.570795 3.14159, axis 1 0 0, limit lower=-2.62 upper=2.62 effort=300 velocity=1
- added joint joint5: type revolute, parent link4, child link5, origin xyz=0.03 0.0 0.0 rpy=0 1.570795 0, axis 1 0 0, limit lower=-2.62 upper=2.62 effort=300 velocity=1
- added joint joint6: type revolute, parent link5, child link6, origin xyz=0 0 0.03 rpy=4.712384999999999 -1.570795 0, axis 1 0 0, limit lower=-6.28 upper=6.28 effort=300 velocity=1

File: unitree_ros-master/robots/aliengo_description/xacro/aliengo1.urdf (robot description, URDF)
Before this commit: robot aliengo_description, 30 links, 29 joints
Links:
- removed link camera
- added link camera_bottom_screw_frame
- added link camera_color_frame
- added link camera_color_optical_frame
- added link camera_depth_frame
- added link camera_depth_optical_frame
- added link camera_left_ir_frame
- added link camera_left_ir_optical_frame
- added link camera_link; collision box size=0.02505 0.09 0.025; visual mesh filename=package://realsense2_description/meshes/d435.dae
- added link camera_right_ir_frame
- added link camera_right_ir_optical_frame
Joints:
- removed joint camera2base_link
- added joint camera_color_joint: type fixed, parent camera_depth_frame, child camera_color_frame, origin xyz=0 0.015 0 rpy=0 0 0
- added joint camera_color_optical_joint: type fixed, parent camera_color_frame, child camera_color_optical_frame, origin xyz=0 0 0 rpy=-1.57079632679 0 -1.57079632679
- added joint camera_depth_joint: type fixed, parent camera_link, child camera_depth_frame, origin xyz=0 0 0 rpy=0 0 0
- added joint camera_depth_optical_joint: type fixed, parent camera_depth_frame, child camera_depth_optical_frame, origin xyz=0 0 0 rpy=-1.57079632679 0 -1.57079632679
- added joint camera_joint: type fixed, parent trunk, child camera_bottom_screw_frame, origin xyz=0.317 0 -0.032 rpy=0 0 0
- added joint camera_left_ir_joint: type fixed, parent camera_depth_frame, child camera_left_ir_frame, origin xyz=0 0.0 0 rpy=0 0 0
- added joint camera_left_ir_optical_joint: type fixed, parent camera_left_ir_frame, child camera_left_ir_optical_frame, origin xyz=0 0 0 rpy=-1.57079632679 0 -1.57079632679
- added joint camera_link_joint: type fixed, parent camera_bottom_screw_frame, child camera_link, origin xyz=0 0.0175 0.0125 rpy=0 0 0
- added joint camera_right_ir_joint: type fixed, parent camera_depth_frame, child camera_right_ir_frame, origin xyz=0 -0.05 0 rpy=0 0 0
- added joint camera_right_ir_optical_joint: type fixed, parent camera_right_ir_frame, child camera_right_ir_optical_frame, origin xyz=0 0 0 rpy=-1.57079632679 0 -1.57079632679
- joint bottom_joint: origin xyz=0 0 -0.025 rpy=0 0 0 -> xyz=0 0 0 rpy=0 0 0

File: unitree_ros-master/robots/aliengo_description/xacro/arm.xacro (robot description, xacro)
@@ -53,5 +53,5 @@
     <!-- ///////////////////////////////////////   bottom_joint   ////////////////////////////////////////// -->
     <joint name="bottom_joint" type="fixed">
-        <origin xyz="0 0 -0.025" rpy="0 0 0" />
+        <origin xyz="0 0 0" rpy="0 0 0" />
         <parent link="trunk"/>
         <child link="bottom_link"/>
@@ -287,13 +287,13 @@
     </joint>
     <!-- /////////////////////////////////   camera   ////////////////////////////////////// -->
-    <xacro:include filename="camera.xacro" />
-    <xacro:include filename="camera_sensor.xacro" />
+    <!-- <xacro:include filename="camera.xacro" /> -->
+    <!-- <xacro:include filename="camera_sensor.xacro" /> -->
     <!-- /////////////////////////////////   Gazebo   ////////////////////////////////////// -->
     <gazebo reference="bottom_link">
         <material>Gazebo/Black</material>
     </gazebo>
-    <gazebo reference="base_link">
-        <material>Gazebo/White</material>
-    </gazebo>
+    <!-- <gazebo reference="base_link">
+        <material>Gazebo/White</material>
+    </gazebo> -->
     <gazebo reference="link1">
         <material>Gazebo/Blue</material>

File: unitree_ros-master/robots/aliengo_description/xacro/robot.xacro (robot description, xacro)
@@ -9,5 +9,5 @@
     <xacro:property name="rolloverProtection" value="false"/>
     <!-- Debug mode will hung up the robot, use "true" or "false" to switch it. -->
-    <!-- <xacro:if value="$(arg DEBUG)">
+    <!-- <xacro:if value="true">
         <link name="world"/>
         <joint name="base_static_joint" type="fixed">
@@ -88,4 +88,213 @@
         </link>
     </xacro:if>
+  <!--
+    ///////////////////////////////////////
+   -->
+  <material name="camera_aluminum">
+    <color rgba="0.5 0.5 0.5 1"/>
+  </material>
+  <joint name="camera_joint" type="fixed">
+    <origin rpy="0 0 0" xyz="0.317 0 -0.032"/>
+    <parent link="trunk"/>
+    <child link="camera_bottom_screw_frame"/>
+  </joint>
+  <link name="camera_bottom_screw_frame"/>
+  <joint name="camera_link_joint" type="fixed">
+    <origin rpy="0 0 0" xyz="0 0.0175 0.0125"/>
+    <parent link="camera_bottom_screw_frame"/>
+    <child link="camera_link"/>
+  </joint>
+  <link name="camera_link">
+    <visual>
+      <origin rpy="1.57079632679 0 1.57079632679" xyz="0.0149 -0.0175 0"/>
+      <geometry>
+        <!-- <box size="0.09 0.025 0.02505"/> -->
+        <mesh filename="package://realsense2_description/meshes/d435.dae"/>
+        <!--<mesh filename="package://realsense2_description/meshes/d435/d435.dae" />-->
+      </geometry>
+      <material name="camera_aluminum"/>
+    </visual>
+    <collision>
+      <origin rpy="0 0 0" xyz="0 -0.0175 0"/>
+      <geometry>
+        <box size="0.02505 0.09 0.025"/>
+      </geometry>
+    </collision>
+  </link>
+  <joint name="camera_depth_joint" type="fixed">
+    <origin rpy="0 0 0" xyz="0 0 0"/>
+    <parent link="camera_link"/>
+    <child link="camera_depth_frame"/>
+  </joint>
+  <link name="camera_depth_frame"/>
+  <joint name="camera_depth_optical_joint" type="fixed">
+    <origin rpy="-1.57079632679 0 -1.57079632679" xyz="0 0 0"/>
+    <parent link="camera_depth_frame"/>
+    <child link="camera_depth_optical_frame"/>
+  </joint>
+  <link name="camera_depth_optical_frame"/>
+  <joint name="camera_left_ir_joint" type="fixed">
+    <origin rpy="0 0 0" xyz="0 0.0 0"/>
+    <parent link="camera_depth_frame"/>
+    <child link="camera_left_ir_frame"/>
+  </joint>
+  <link name="camera_left_ir_frame"/>
+  <joint name="camera_left_ir_optical_joint" type="fixed">
+    <origin rpy="-1.57079632679 0 -1.57079632679" xyz="0 0 0"/>
+    <parent link="camera_left_ir_frame"/>
+    <child link="camera_left_ir_optical_frame"/>
+  </joint>
+  <link name="camera_left_ir_optical_frame"/>
+  <joint name="camera_right_ir_joint" type="fixed">
+    <origin rpy="0 0 0" xyz="0 -0.05 0"/>
+    <parent link="camera_depth_frame"/>
+    <child link="camera_right_ir_frame"/>
+  </joint>
+  <link name="camera_right_ir_frame"/>
+  <joint name="camera_right_ir_optical_joint" type="fixed">
+    <origin rpy="-1.57079632679 0 -1.57079632679" xyz="0 0 0"/>
+    <parent link="camera_right_ir_frame"/>
+    <child link="camera_right_ir_optical_frame"/>
+  </joint>
+  <link name="camera_right_ir_optical_frame"/>
+  <joint name="camera_color_joint" type="fixed">
+    <origin rpy="0 0 0" xyz="0 0.015 0"/>
+    <parent link="camera_depth_frame"/>
+    <child link="camera_color_frame"/>
+  </joint>
+  <link name="camera_color_frame"/>
+  <joint name="camera_color_optical_joint" type="fixed">
+    <origin rpy="-1.57079632679 0 -1.57079632679" xyz="0 0 0"/>
+    <parent link="camera_color_frame"/>
+    <child link="camera_color_optical_frame"/>
+  </joint>
+  <link name="camera_color_optical_frame"/>
+  <gazebo reference="camera_link">
+    <self_collide>0</self_collide>
+    <enable_wind>0</enable_wind>
+    <kinematic>0</kinematic>
+    <gravity>1</gravity>
+    <!--<mu>1</mu>-->
+    <mu2>1</mu2>
+    <fdir1>0 0 0</fdir1>
+    <!--<slip1>0</slip1>
+      <slip2>0</slip2>-->
+    <kp>1e+13</kp>
+    <kd>1</kd>
+    <!--<max_vel>0.01</max_vel>
+      <min_depth>0</min_depth>-->
+    <sensor name="cameracolor" type="camera">
+      <camera name="camera">
+        <horizontal_fov>1.5</horizontal_fov>
+        <image>
+          <width>1280</width>
+          <height>720</height>
+          <format>RGB_INT8</format>
+        </image>
+        <clip>
+          <near>0.1</near>
+          <far>100</far>
+        </clip>
+        <noise>
+          <type>gaussian</type>
+          <mean>0.0</mean>
+          <stddev>0.007</stddev>
+        </noise>
+      </camera>
+      <always_on>1</always_on>
+      <update_rate>30</update_rate>
+      <visualize>0</visualize>
+    </sensor>
+    <sensor name="cameraired1" type="camera">
+      <camera name="camera">
+        <horizontal_fov>1.4870205227</horizontal_fov>
+        <image>
+          <width>1280</width>
+          <height>720</height>
+          <format>L_INT8</format>
+        </image>
+        <clip>
+          <near>0.1</near>
+          <far>100</far>
+        </clip>
+        <noise>
+          <type>gaussian</type>
+          <mean>0.0</mean>
+          <stddev>0.05</stddev>
+        </noise>
+      </camera>
+      <always_on>0</always_on>
+      <update_rate>90</update_rate>
+      <visualize>0</visualize>
+    </sensor>
+    <sensor name="cameraired2" type="camera">
+      <camera name="camera">
+        <horizontal_fov>1.4870205227</horizontal_fov>
+        <image>
+          <width>1280</width>
+          <height>720</height>
+          <format>L_INT8</format>
+        </image>
+        <clip>
+          <near>0.1</near>
+          <far>100</far>
+        </clip>
+        <noise>
+          <type>gaussian</type>
+          <mean>0.0</mean>
+          <stddev>0.05</stddev>
+        </noise>
+      </camera>
+      <always_on>0</always_on>
+      <update_rate>90</update_rate>
+      <visualize>0</visualize>
+    </sensor>
+    <sensor name="cameradepth" type="depth">
+      <camera name="camera">
+        <horizontal_fov>1.5</horizontal_fov>
+        <image>
+          <width>1280</width>
+          <height>720</height>
+        </image>
+        <clip>
+          <near>0.1</near>
+          <far>100</far>
+        </clip>
+        <noise>
+          <type>gaussian</type>
+          <mean>0.0</mean>
+          <stddev>0.100</stddev>
+        </noise>
+      </camera>
+      <always_on>1</always_on>
+      <update_rate>90</update_rate>
+      <visualize>0</visualize>
+    </sensor>
+  </gazebo>
+  <gazebo>
+    <plugin filename="librealsense_gazebo_plugin.so" name="camera">
+      <prefix>camera</prefix>
+      <depthUpdateRate>30.0</depthUpdateRate>
+      <colorUpdateRate>30.0</colorUpdateRate>
+      <infraredUpdateRate>30.0</infraredUpdateRate>
+      <depthTopicName>depth/image_raw</depthTopicName>
+      <depthCameraInfoTopicName>depth/camera_info</depthCameraInfoTopicName>
+      <colorTopicName>color/image_raw</colorTopicName>
+      <colorCameraInfoTopicName>color/camera_info</colorCameraInfoTopicName>
+      <infrared1TopicName>infra1/image_raw</infrared1TopicName>
+      <infrared1CameraInfoTopicName>infra1/camera_info</infrared1CameraInfoTopicName>
+      <infrared2TopicName>infra2/image_raw</infrared2TopicName>
+      <infrared2CameraInfoTopicName>infra2/camera_info</infrared2CameraInfoTopicName>
+      <colorOpticalframeName>camera_depth_optical_frame</colorOpticalframeName>
+      <depthOpticalframeName>camera_depth_optical_frame</depthOpticalframeName>
+      <infrared1OpticalframeName>camera_left_ir_optical_frame</infrared1OpticalframeName>
+      <infrared2OpticalframeName>camera_right_ir_optical_frame</infrared2OpticalframeName>
+      <rangeMinDepth>0.28</rangeMinDepth>
+      <rangeMaxDepth>10.0</rangeMaxDepth>
+    </plugin>
+  </gazebo>
+  <!--
+    ///////////////////////////////////////////////////
+   -->
     <joint name="imu_joint" type="fixed">
         <parent link="trunk"/>

Commit message: final nav

File: unitree_ros-master/robots/aliengo_description/xacro/aliengo.urdf (robot description, URDF)
Before this commit: robot aliengo_description, 39 links, 38 joints
Links:
- removed link grasping_frame
- added link camera, mass 0.01; collision box size=0.001 0.01 0.01; visual box size=0.001 0.01 0.01
- link bottom_link: mass 0.2 -> 0.1
- link gripper_finger_link1: mass 0.2 -> 0.1; geometry collision box size=0.06 0.01 0.01; visual box size=0.06 0.01 0.01
- link gripper_finger_link2: mass 0.2 -> 0.1; geometry collision box size=0.06 0.01 0.01; visual box size=0.06 0.01 0.01
- link link1: mass 0.2 -> 0.1; geometry collision cylinder length=0.015 radius=0.003; visual cylinder length=0.15 radius=0.03
- link link2: mass 0.2 -> 0.1; geometry collision cylinder length=0.02 radius=0.003; visual cylinder length=0.2 radius=0.03
- link link3: mass 0.2 -> 0.1; geometry collision cylinder length=0.02 radius=0.003; visual cylinder length=0.2 radius=0.03
- link link4: mass 0.2 -> 0.1
- link link5: mass 0.2 -> 0.1
- link link6: mass 0.2 -> 0.1
Joints:
- removed joint grasping_frame_joint
- added joint camera2base_link: type fixed, parent link6, child camera, origin xyz=0.0205 0.0 0.0 rpy=3.1416 0.0 0.0
- joint bottom_joint: origin xyz=0 0 0 rpy=0 0 0 -> xyz=0.15 0 -0.025 rpy=0 0 0
- joint joint1: axis -1 0 0 -> 1 0 0; parent trunk -> bottom_link
- joint joint3: origin xyz=0 0 0.22 rpy=0 3.14159 0 -> xyz=0 0 0.2 rpy=0 3.14159 0
- joint joint4: origin xyz=0.0 0.0 -0.14 rpy=0 1.570795 3.14159 -> xyz=0.0 0.0 -0.2 rpy=0 1.570795 3.14159
- joint joint5: axis 1 0 0 -> -1 0 0
